Commit message: RPP controller

File: src/mtu28_jackal/mtu28_description/urdf/zedgnssfusion_mtu28_jackal_description.urdf.xacro (robot description, xacro)
@@ -10,5 +10,5 @@
   <xacro:arg name="gnss_z" default="0.197" />
   <xacro:arg name="use_zed_localization" default="false" /> <!-- odom frame to camera_link frame if true -->
-  <xacro:arg name="parent_link" default="fath_pivot_0_mount" />  <!-- only when use_zed_localization is false-->
+  <xacro:arg name="parent_link" default="base_link" />  <!-- only when use_zed_localization is false-->
   <xacro:include filename="$(find project_description)/urdf/zed_macro.urdf.xacro" />
   <xacro:zed_camera name="$(arg camera_name)"
@@ -22,5 +22,5 @@
                     gnss_z="$(arg gnss_z)">
        <!-- when use_zed_localization is false, this should provide the transform from the mount to the camera_link -->
-      <origin xyz="0.0 0.0 0.0" rpy="0 0 0"/>
+      <origin xyz="0.252 0.0 0.226" rpy="0 0 0"/>
       <!-- camera link to base_link when use_zed_localization is true -->
       <!-- <origin xyz="-0.252 0.000 -0.226" rpy="0 0 0"/>        -->
